Commit message: Delete redundant lines.

File: ahl_robot/youbot/virtual_youbot/ahl_youbot_description/urdf/arm/arm.urdf.xacro (robot description, xacro)
@@ -7,5 +7,5 @@
   <xacro:include filename="$(find ahl_youbot_description)/urdf/arm/arm.transmission.xacro" />
   <xacro:include filename="$(find ahl_youbot_description)/urdf/arm/limits.urdf.xacro" />
-  <xacro:macro name="youbot_arm" params="parent name *origin">
+  <xacro:macro name="youbot_arm" params="name">
     <!-- joint between base_link and arm_0_link -->
     <joint name="${name}_joint_0" type="fixed" >
@@ -168,6 +168,6 @@
     </link>
     <!-- extensions -->
-    <xacro:youbot_arm_gazebo name="${name}" />
-    <xacro:youbot_arm_transmission name="${name}" />
+    <xacro:youbot_arm_gazebo name="${name}"/>
+    <xacro:youbot_arm_transmission name="${name}"/>
   </xacro:macro>
 </robot>

File: ahl_robot/youbot/virtual_youbot/ahl_youbot_description/urdf/gripper/gripper.urdf.xacro (robot description, xacro)
@@ -7,9 +7,9 @@
   <xacro:include filename="$(find youbot_description)/urdf/youbot_gripper/gripper.transmission.xacro" />
   <xacro:include filename="$(find youbot_description)/urdf/youbot_gripper/limits.urdf.xacro" />
-  <xacro:macro name="youbot_gripper" params="parent name *origin">
+  <xacro:macro name="youbot_gripper" params="name">
     <!-- joint between arm_7_link and sdh_palm_link -->
     <joint name="${name}_palm_joint" type="fixed" >
-      <insert_block name="origin"/>
-      <parent link="${parent}" />
+      <origin xyz="0 0 0.04" rpy="0 0 0"/>
+      <parent link="arm_link_5" />
       <child link="${name}_palm_link" />
     </joint>

File: ahl_robot/youbot/virtual_youbot/ahl_youbot_description/urdf/youbot.urdf.xacro (robot description, xacro)
@@ -13,10 +13,6 @@
   <xacro:include filename="$(find ahl_youbot_description)/controller/ros_controller.urdf.xacro" />
 -->
-  <xacro:youbot_base name="base"/>
-  <xacro:youbot_arm name="arm" parent="base_link">
-    <origin xyz="0.143 0 0.046" rpy="0 0 0" />
-  </xacro:youbot_arm>
-  <xacro:youbot_gripper name="gripper" parent="arm_link_5">
-    <origin xyz="0 0 0.04" rpy="0 0 0"/>
-  </xacro:youbot_gripper>
+  <xacro:youbot_base    name="base"/>
+  <xacro:youbot_arm     name="arm"/>
+  <xacro:youbot_gripper name="gripper"/>
 </robot>

Commit message: Deleted unnecessary spaces.

File: ahl_robot/youbot/virtual_youbot/ahl_youbot_description/urdf/arm/arm.urdf.xacro (robot description, xacro)
@@ -4,21 +4,21 @@
         xmlns:interface="http://playerstage.sourceforge.net/gazebo/xmlschema/#interface"
         xmlns:xacro="http://ros.org/wiki/xacro">
-  <xacro:include filename="$(find ahl_youbot_description)/urdf/arm/arm.gazebo.xacro" />
-  <xacro:include filename="$(find ahl_youbot_description)/urdf/arm/arm.transmission.xacro" />
-  <xacro:include filename="$(find ahl_youbot_description)/urdf/arm/limits.urdf.xacro" />
+  <xacro:include filename="$(find ahl_youbot_description)/urdf/arm/arm.gazebo.xacro"/>
+  <xacro:include filename="$(find ahl_youbot_description)/urdf/arm/arm.transmission.xacro"/>
+  <xacro:include filename="$(find ahl_youbot_description)/urdf/arm/limits.urdf.xacro"/>
   <xacro:macro name="youbot_arm" params="name">
     <!-- joint between base_link and arm_0_link -->
-    <joint name="${name}_joint_0" type="fixed" >
+    <joint name="${name}_joint_0" type="fixed">
       <origin xyz="0.143 0 0.0207" rpy="0 0 0"/>
-      <parent link="base_link" />
-      <child  link="${name}_link_0" />
+      <parent link="base_link"/>
+      <child  link="${name}_link_0"/>
     </joint>
     <link name="${name}_link_0">
       <inertial>
         <mass value="${link_0_mass}"/>
-        <xacro:link_0_inertia_tensor />
+        <xacro:link_0_inertia_tensor/>
       </inertial>
       <visual>
-        <origin xyz="0 0 0.0318" rpy="0 0 0" />
+        <origin xyz="0 0 0.0318" rpy="0 0 0"/>
         <geometry>
           <mesh filename="package://ahl_youbot_description/meshes/arm/arm0.dae"/>
@@ -38,5 +38,5 @@
       <child link="${name}_link_1"/>
       <axis xyz="0 0 1"/>
-      <dynamics damping="0.1" friction="0" />
+      <dynamics damping="0.1" friction="0"/>
       <limit effort="9.5" velocity="2.5" lower="${joint_1_lower_limit}" upper="${joint_1_upper_limit}"/>
     </joint>
@@ -44,16 +44,16 @@
       <inertial>
         <mass value="${link_1_mass}"/>
-        <xacro:link_1_inertia_tensor />
+        <xacro:link_1_inertia_tensor/>
       </inertial>
       <visual>
-        <origin xyz="0 0 0.0499" rpy="0 0 0" />
+        <origin xyz="0 0 0.0499" rpy="0 0 0"/>
         <geometry>
-          <mesh filename="package://ahl_youbot_description/meshes/arm/arm1.dae" />
+          <mesh filename="package://ahl_youbot_description/meshes/arm/arm1.dae"/>
         </geometry>
       </visual>
       <collision>
-        <origin xyz="0 0 0.0499" rpy="0 0 0" />
+        <origin xyz="0 0 0.0499" rpy="0 0 0"/>
         <geometry>
-          <mesh filename="package://ahl_youbot_description/meshes/arm/arm1_convex.stl" />
+          <mesh filename="package://ahl_youbot_description/meshes/arm/arm1_convex.stl"/>
         </geometry>
       </collision>
@@ -74,7 +74,7 @@
       </inertial>
       <visual>
-        <origin xyz="0 -0.032 0.078" rpy="0 0 0" />
+        <origin xyz="0 -0.032 0.078" rpy="0 0 0"/>
         <geometry>
-          <mesh filename="package://ahl_youbot_description/meshes/arm/arm2.dae" />
+          <mesh filename="package://ahl_youbot_description/meshes/arm/arm2.dae"/>
         </geometry>
       </visual>
@@ -92,5 +92,5 @@
       <child link="${name}_link_3"/>
       <axis xyz="0 1 0"/>
-      <dynamics damping="0.1" friction="0" />
+      <dynamics damping="0.1" friction="0"/>
       <limit effort="6.0" velocity="2.5" lower="${joint_3_lower_limit}" upper="${joint_3_upper_limit}"/>
     </joint>
@@ -98,16 +98,16 @@
       <inertial>
         <mass value="${link_3_mass}"/>
-        <xacro:link_3_inertia_tensor />
+        <xacro:link_3_inertia_tensor/>
       </inertial>
       <visual>
-        <origin xyz="0.000 0.028 0.079" rpy="0 0 0" />
+        <origin xyz="0.000 0.028 0.079" rpy="0 0 0"/>
         <geometry>
-          <mesh filename="package://ahl_youbot_description/meshes/arm/arm3.dae" />
+          <mesh filename="package://ahl_youbot_description/meshes/arm/arm3.dae"/>
         </geometry>
       </visual>
       <collision>
-        <origin xyz="0.000 0.028 0.079" rpy="0 0 0" />
+        <origin xyz="0.000 0.028 0.079" rpy="0 0 0"/>
         <geometry>
-          <mesh filename="package://ahl_youbot_description/meshes/arm/arm3_convex.stl" />
+          <mesh filename="package://ahl_youbot_description/meshes/arm/arm3_convex.stl"/>
         </geometry>
       </collision>
@@ -115,9 +115,9 @@
     <!-- joint between arm_3_link and arm_4_link -->
     <joint name="${name}_joint_4" type="revolute">
-      <origin xyz="0.000 0.000 0.135" rpy="0 0 0" />
+      <origin xyz="0.000 0.000 0.135" rpy="0 0 0"/>
       <parent link="${name}_link_3"/>
       <child link="${name}_link_4"/>
-      <axis xyz="0 1 0" />
-      <dynamics damping="0.1" friction="0" />
+      <axis xyz="0 1 0"/>
+      <dynamics damping="0.1" friction="0"/>
       <limit effort="2.0" velocity="1.5" lower="${joint_4_lower_limit}" upper="${joint_4_upper_limit}"/>
     </joint>
@@ -125,10 +125,10 @@
       <inertial>
         <mass value="${link_4_mass}"/>
-        <xacro:link_4_inertia_tensor />
+        <xacro:link_4_inertia_tensor/>
       </inertial>
       <visual>
         <origin xyz="0 -0.010 0.029" rpy="0 0 0"/>
         <geometry>
-          <mesh filename="package://ahl_youbot_description/meshes/arm/arm4.dae" />
+          <mesh filename="package://ahl_youbot_description/meshes/arm/arm4.dae"/>
         </geometry>
       </visual>
@@ -136,5 +136,5 @@
         <origin xyz="0 -0.010 0.029" rpy="0 0 0"/>
         <geometry>
-          <mesh filename="package://ahl_youbot_description/meshes/arm/arm4_convex.stl" />
+          <mesh filename="package://ahl_youbot_description/meshes/arm/arm4_convex.stl"/>
         </geometry>
       </collision>
@@ -142,26 +142,26 @@
     <!-- joint between arm_4_link and arm_5_link -->
     <joint name="${name}_joint_5" type="revolute">
-      <origin xyz="0 0 0.084" rpy="0 0 0" />
+      <origin xyz="0 0 0.084" rpy="0 0 0"/>
       <parent link="${name}_link_4"/>
       <child link="${name}_link_5"/>
-      <axis xyz="0 0 1" />
-      <dynamics damping="0.1" friction="0" />
-      <limit effort="1.0" velocity="1.5" lower="${joint_5_lower_limit}" upper="${joint_5_upper_limit}" />
+      <axis xyz="0 0 1"/>
+      <dynamics damping="0.1" friction="0"/>
+      <limit effort="1.0" velocity="1.5" lower="${joint_5_lower_limit}" upper="${joint_5_upper_limit}"/>
     </joint>
     <link name="${name}_link_5">
       <inertial>
         <mass value="${link_5_mass}"/>
-        <xacro:link_5_inertia_tensor />
+        <xacro:link_5_inertia_tensor/>
       </inertial>
       <visual>
-        <origin xyz="0 0 0.0188" rpy="0 0 0" />
+        <origin xyz="0 0 0.0188" rpy="0 0 0"/>
         <geometry>
-          <mesh filename="package://ahl_youbot_description/meshes/arm/arm5.dae" />
+          <mesh filename="package://ahl_youbot_description/meshes/arm/arm5.dae"/>
         </geometry>
       </visual>
       <collision>
-        <origin xyz="0 0 0.0188" rpy="0 0 0" />
+        <origin xyz="0 0 0.0188" rpy="0 0 0"/>
         <geometry>
-          <mesh filename="package://ahl_youbot_description/meshes/arm/arm5_convex.stl" />
+          <mesh filename="package://ahl_youbot_description/meshes/arm/arm5_convex.stl"/>
         </geometry>
       </collision>

File: ahl_robot/youbot/virtual_youbot/ahl_youbot_description/urdf/arm/limits.urdf.xacro (robot description, xacro)
@@ -6,52 +6,52 @@
   <!-- arm limits positions (deg) -->
   <property name="joint_1_lower_limit" value="-${M_PI * 169 / 180}"/>
-  <property name="joint_1_upper_limit" value="${M_PI * 169 / 180}"/>
-  <property name="joint_2_lower_limit" value="-${M_PI * 65 / 180}"/>
-  <property name="joint_2_upper_limit" value="${M_PI * 90 / 180}"/>
+  <property name="joint_1_upper_limit" value= "${M_PI * 169 / 180}"/>
+  <property name="joint_2_lower_limit" value="-${M_PI *  65 / 180}"/>
+  <property name="joint_2_upper_limit" value= "${M_PI *  90 / 180}"/>
   <property name="joint_3_lower_limit" value="-${M_PI * 151 / 180}"/>
-  <property name="joint_3_upper_limit" value="${M_PI * 146 / 180}"/>
+  <property name="joint_3_upper_limit" value= "${M_PI * 146 / 180}"/>
   <property name="joint_4_lower_limit" value="-${M_PI * 102.5 / 180}"/>
-  <property name="joint_4_upper_limit" value="${M_PI * 102.5 / 180}"/>
+  <property name="joint_4_upper_limit" value= "${M_PI * 102.5 / 180}"/>
   <property name="joint_5_lower_limit" value="-${M_PI * 165 / 180}"/>
-  <property name="joint_5_upper_limit" value="${M_PI * 165 / 180}"/>
+  <property name="joint_5_upper_limit" value= "${M_PI * 165 / 180}"/>
   <property name="joint_1_lower_limit_soft" value="-${(M_PI * 169 / 180) + threshold}"/>
-  <property name="joint_1_upper_limit_soft" value="${(M_PI * 169 / 180) - threshold}"/>
-  <property name="joint_2_lower_limit_soft" value="-${(M_PI * 65 / 180) + threshold}"/>
-  <property name="joint_2_upper_limit_soft" value="${(M_PI * 90 / 180) - threshold}"/>
+  <property name="joint_1_upper_limit_soft" value= "${(M_PI * 169 / 180) - threshold}"/>
+  <property name="joint_2_lower_limit_soft" value="-${(M_PI *  65 / 180) + threshold}"/>
+  <property name="joint_2_upper_limit_soft" value= "${(M_PI *  90 / 180) - threshold}"/>
   <property name="joint_3_lower_limit_soft" value="-${(M_PI * 151 / 180) + threshold}"/>
-  <property name="joint_3_upper_limit_soft" value="${(M_PI * 146 / 180) - threshold}"/>
+  <property name="joint_3_upper_limit_soft" value= "${(M_PI * 146 / 180) - threshold}"/>
   <property name="joint_4_lower_limit_soft" value="-${(M_PI * 102.5 / 180) + threshold}"/>
-  <property name="joint_4_upper_limit_soft" value="${(M_PI * 102.5 / 180) - threshold}"/>
+  <property name="joint_4_upper_limit_soft" value= "${(M_PI * 102.5 / 180) - threshold}"/>
   <property name="joint_5_lower_limit_soft" value="-${(M_PI * 165 / 180) + threshold}"/>
-  <property name="joint_5_upper_limit_soft" value="${(M_PI * 165 / 180) - threshold}"/>
+  <property name="joint_5_upper_limit_soft" value= "${(M_PI * 165 / 180) - threshold}"/>
   <!-- dynamic properties : mass (kg) Alu data sheet -->
-  <property name="link_0_mass" value="0.961" />
-  <property name="link_1_mass" value="1.390" />
-  <property name="link_2_mass" value="1.318" />
-  <property name="link_3_mass" value="0.821" />
-  <property name="link_4_mass" value="0.769" />
-  <property name="link_5_mass" value="0.687" />
+  <property name="link_0_mass" value="0.961"/>
+  <property name="link_1_mass" value="1.390"/>
+  <property name="link_2_mass" value="1.318"/>
+  <property name="link_3_mass" value="0.821"/>
+  <property name="link_4_mass" value="0.769"/>
+  <property name="link_5_mass" value="0.687"/>
   <xacro:macro name="link_0_inertia_tensor">
-    <origin xyz="0.015221 -0.000041 0.033843" rpy="0 0 0" />
+    <origin xyz="0.015221 -0.000041 0.033843" rpy="0 0 0"/>
     <inertia ixx="0.001875" ixy="0" ixz="0" iyy="0.001875" iyz="0" izz="0.002775"/>
   </xacro:macro>
   <xacro:macro name="link_1_inertia_tensor">
-    <origin xyz="-0.010838 0.006337 0.034345" rpy="0 0 0" />
+    <origin xyz="-0.010838 0.006337 0.034345" rpy="0 0 0"/>
     <inertia ixx="0.003003" ixy="0" ixz="0" iyy="0.003003" iyz="0" izz="0.004904"/>
   </xacro:macro>
   <xacro:macro name="link_2_inertia_tensor">
-    <origin xyz="0.001377 -0.029369 0.086325" rpy="0 0 0" />
+    <origin xyz="0.001377 -0.029369 0.086325" rpy="0 0 0"/>
     <inertia ixx="0.0031631" ixy="0" ixz="0" iyy="0.0031145" iyz="0" izz="0.0005843"/>
   </xacro:macro>
   <xacro:macro name="link_3_inertia_tensor">
-    <origin xyz="0.000130 0.028599 0.079400" rpy="0 0 0" />
+    <origin xyz="0.000130 0.028599 0.079400" rpy="0 0 0"/>
     <inertia ixx="0.0018468" ixy="0" ixz="0" iyy="0.00172767" iyz="0" izz="0.0005843"/>
   </xacro:macro>
   <xacro:macro name="link_4_inertia_tensor">
-    <origin xyz="0.000124 -0.005595 0.040469" rpy="0 0 0"  />
+    <origin xyz="0.000124 -0.005595 0.040469" rpy="0 0 0"/>
     <inertia ixx="0.0010573" ixy="0" ixz="0" iyy="0.0006764" iyz="0" izz="0.0006610"/>
   </xacro:macro>
   <xacro:macro name="link_5_inertia_tensor">
-    <origin xyz="-0.000903 0.000638 0.006573" rpy="0 0 0" />
+    <origin xyz="-0.000903 0.000638 0.006573" rpy="0 0 0"/>
     <inertia ixx="0.0001602" ixy="0" ixz="0" iyy="0.0000689" iyz="0" izz="0.0001934"/>
   </xacro:macro>

File: ahl_robot/youbot/virtual_youbot/ahl_youbot_description/urdf/base/base.transmission.xacro (robot description, xacro)
@@ -4,7 +4,6 @@
        xmlns:interface="http://playerstage.sourceforge.net/gazebo/xmlschema/#interface"
        xmlns:xacro="http://ros.org/wiki/xacro">
-  <property name="wheel_mechanical_reduction" value="${624/35 * 80/18}" />
-  <property name="caster_mechanical_reduction" value="${624/35 * 80/18}" />
-  <property name="" value="0.360" />
+  <property name="wheel_mechanical_reduction" value="${624/35 * 80/18}"/>
+  <property name="caster_mechanical_reduction" value="${624/35 * 80/18}"/>
   <xacro:macro name="youbot_base_transmission">
   <!-- front left wheel -->

File: ahl_robot/youbot/virtual_youbot/ahl_youbot_description/urdf/base/base.urdf.xacro (robot description, xacro)
@@ -13,5 +13,4 @@
   <property name="caster_offset_x" value="0.228"/>
   <property name="caster_offset_y" value="0.158"/>
-<!--  <property name="caster_offset_z" value="-0.034"/> -->
   <property name="caster_offset_z" value="-0.0463"/>
   <property name="caster_mass" value="0.001"/>
@@ -65,5 +64,4 @@
         <origin xyz="0 0 0" rpy="0 0 0"/>
         <geometry>
-          <!--<box size="${base_size_x} ${base_size_y} ${base_size_z}" />-->
           <mesh filename="package://ahl_youbot_description/meshes/base/base_convex.stl"/>
         </geometry>
@@ -252,5 +250,4 @@
     <joint name="plate_joint" type="fixed">
       <origin xyz="${plate_offset_x} ${plate_offset_y} ${plate_offset_z}" rpy="0 0 0"/>
-<!-- <parent link="${name}_link"/>-->
       <parent link="base_link"/>
       <child link="plate_link"/>

File: ahl_robot/youbot/virtual_youbot/ahl_youbot_description/urdf/gripper/gripper.urdf.xacro (robot description, xacro)
@@ -4,13 +4,13 @@
        xmlns:interface="http://playerstage.sourceforge.net/gazebo/xmlschema/#interface"
        xmlns:xacro="http://ros.org/wiki/xacro">
-  <xacro:include filename="$(find youbot_description)/urdf/youbot_gripper/gripper.gazebo.xacro" />
-  <xacro:include filename="$(find youbot_description)/urdf/youbot_gripper/gripper.transmission.xacro" />
-  <xacro:include filename="$(find youbot_description)/urdf/youbot_gripper/limits.urdf.xacro" />
+  <xacro:include filename="$(find youbot_description)/urdf/youbot_gripper/gripper.gazebo.xacro"/>
+  <xacro:include filename="$(find youbot_description)/urdf/youbot_gripper/gripper.transmission.xacro"/>
+  <xacro:include filename="$(find youbot_description)/urdf/youbot_gripper/limits.urdf.xacro"/>
   <xacro:macro name="youbot_gripper" params="name">
     <!-- joint between arm_7_link and sdh_palm_link -->
-    <joint name="${name}_palm_joint" type="fixed" >
+    <joint name="${name}_palm_joint" type="fixed">
       <origin xyz="0 0 0.04" rpy="0 0 0"/>
-      <parent link="arm_link_5" />
-      <child link="${name}_palm_link" />
+      <parent link="arm_link_5"/>
+      <child link="${name}_palm_link"/>
     </joint>
     <link name="${name}_palm_link">
@@ -18,8 +18,8 @@
         <origin xyz="0.002737 0 0.02616" rpy="0 0 0"/>
         <mass value="0.199"/>
-        <inertia ixx="0.0003629" ixy="0" ixz="0" iyy="0.0002067" iyz="0" izz="0.0002324" />
+        <inertia ixx="0.0003629" ixy="0" ixz="0" iyy="0.0002067" iyz="0" izz="0.0002324"/>
       </inertial>
       <visual>
-        <origin xyz="-0.00273 0 0.0224" rpy="0 0 0" />
+        <origin xyz="-0.00273 0 0.0224" rpy="0 0 0"/>
         <geometry>
           <mesh filename="package://ahl_youbot_description/meshes/gripper/palm.dae"/>
@@ -28,7 +28,7 @@
       </visual>
       <collision>
-        <origin xyz="-0.00273 0 0.0224" rpy="0 0 0" />
+        <origin xyz="-0.00273 0 0.0224" rpy="0 0 0"/>
         <geometry>
-          <mesh filename="package://ahl_youbot_description/meshes/gripper/palm_convex.stl" />
+          <mesh filename="package://ahl_youbot_description/meshes/gripper/palm_convex.stl"/>
         </geometry>
       </collision>
@@ -65,6 +65,6 @@
       <parent link="${name}_palm_link"/>
       <child link="${name}_finger_link_r"/>
-      <axis xyz="0 1 0" />
-      <dynamics damping="5.0" friction="0.5" />
+      <axis xyz="0 1 0"/>
+      <dynamics damping="5.0" friction="0.5"/>
       <limit effort="0.5" velocity="0.1" lower="-${finger_joint}" upper="0"/>
     </joint>
@@ -73,5 +73,5 @@
         <origin xyz="0.000270 -0.001337 0.020234" rpy="0 0 0"/>
         <mass value="0.01"/>
-        <inertia ixx="0" ixy="0" ixz="0" iyy="0" iyz="0" izz="0" />
+        <inertia ixx="0" ixy="0" ixz="0" iyy="0" iyz="0" izz="0"/>
       </inertial>
       <visual>
@@ -89,6 +89,6 @@
     </link>
     <!-- extensions -->
-    <xacro:youbot_gripper_gazebo name="${name}" />
-    <xacro:youbot_gripper_transmission name="${name}" />
+    <xacro:youbot_gripper_gazebo name="${name}"/>
+    <xacro:youbot_gripper_transmission name="${name}"/>
   </xacro:macro>
 </robot>

Commit message: Fixed bug. joint_1_***_limit -> joint_2_***_limit

File: ahl_robot/youbot/virtual_youbot/ahl_youbot_description/urdf/arm/arm.urdf.xacro (robot description, xacro)
@@ -66,5 +66,5 @@
       <axis xyz="0 1 0"/>
       <dynamics damping="0.1" friction="0" />
-      <limit effort="9.5" velocity="2.5" lower="${joint_1_lower_limit}" upper="${joint_1_upper_limit}"/>
+      <limit effort="9.5" velocity="2.5" lower="${joint_2_lower_limit}" upper="${joint_2_upper_limit}"/>
     </joint>
     <link name="${name}_link_2">
