Commit message: Added damping to joint and set friction and some gazebo parameters in arm.gazebo.xacro.

File: ahl_robot/youbot/virtual_youbot/ahl_youbot_description/urdf/arm/arm.gazebo.xacro (robot description, xacro)
@@ -6,170 +6,68 @@
   <xacro:macro name="arm_gazebo" params="name">
     <gazebo reference="${name}_link_0">
-      <turnGravityOff>false</turnGravityOff>
-      <surface>
-        <friction>
-          <ode>
-            <mu>0</mu>
-            <mu2>0</mu2>
-            <fdir1>0 0 0</fdir1>
-            <slip1>0</slip1>
-            <slip2>0</slip2>
-	  </ode>
-        </friction>
-        <bounce>
-          <restitution_coefficient>0</restitution_coefficient>
-          <threshold>0</threshold>
-        </bounce>
-        <contact>
-          <ode>
-            <soft_cfm>0</soft_cfm>
-            <soft_erp>0.200000</soft_erp>
-            <kp>10000000000000.000000</kp>
-            <kd>100000000000.000000</kd>
-            <max_vel>-1</max_vel>
-            <min_depth>0</min_depth>
-          </ode>
-        </contact>
-      </surface>
+      <gravity>true</gravity>
+      <maxVel>-1</maxVel>
+      <minDepth>0</minDepth>
+      <mu1>0.3</mu1>
+      <mu2>0.3</mu2>
+      <fdir1></fdir1>
+      <kp>1000000.0</kp>
+      <kd>10000.0</kd>
+      <selfCollide>true</selfCollide>
     </gazebo>
     <gazebo reference="${name}_link_1">
-      <turnGravityOff>false</turnGravityOff>
-      <surface>
-        <friction>
-          <ode>
-            <mu>0</mu>
-            <mu2>0</mu2>
-            <fdir1>0 0 0</fdir1>
-            <slip1>0</slip1>
-            <slip2>0</slip2>
-	  </ode>
-        </friction>
-        <bounce>
-          <restitution_coefficient>0</restitution_coefficient>
-          <threshold>0</threshold>
-        </bounce>
-        <contact>
-          <ode>
-            <soft_cfm>0</soft_cfm>
-            <soft_erp>0.200000</soft_erp>
-            <kp>10000000000000.000000</kp>
-            <kd>100000000000.000000</kd>
-            <max_vel>-1</max_vel>
-            <min_depth>0</min_depth>
-          </ode>
-        </contact>
-      </surface>
+      <gravity>true</gravity>
+      <maxVel>-1</maxVel>
+      <minDepth>0</minDepth>
+      <mu1>0.3</mu1>
+      <mu2>0.3</mu2>
+      <fdir1></fdir1>
+      <kp>1000000.0</kp>
+      <kd>10000.0</kd>
+      <selfCollide>true</selfCollide>
     </gazebo>
     <gazebo reference="${name}_link_2">
-      <turnGravityOff>false</turnGravityOff>
-      <surface>
-        <friction>
-          <ode>
-            <mu>0</mu>
-            <mu2>0</mu2>
-            <fdir1>0 0 0</fdir1>
-            <slip1>0</slip1>
-            <slip2>0</slip2>
-	  </ode>
-        </friction>
-        <bounce>
-          <restitution_coefficient>0</restitution_coefficient>
-          <threshold>0</threshold>
-        </bounce>
-        <contact>
-          <ode>
-            <soft_cfm>0</soft_cfm>
-            <soft_erp>0.200000</soft_erp>
-            <kp>10000000000000.000000</kp>
-            <kd>100000000000.000000</kd>
-            <max_vel>-1</max_vel>
-            <min_depth>0</min_depth>
-          </ode>
-        </contact>
-      </surface>
+      <gravity>true</gravity>
+      <maxVel>-1</maxVel>
+      <minDepth>0</minDepth>
+      <mu1>0.3</mu1>
+      <mu2>0.3</mu2>
+      <fdir1></fdir1>
+      <kp>1000000.0</kp>
+      <kd>10000.0</kd>
+      <selfCollide>true</selfCollide>
     </gazebo>
     <gazebo reference="${name}_link_3">
-      <turnGravityOff>false</turnGravityOff>
-      <surface>
-        <friction>
-          <ode>
-            <mu>0</mu>
-            <mu2>0</mu2>
-            <fdir1>0 0 0</fdir1>
-            <slip1>0</slip1>
-            <slip2>0</slip2>
-	  </ode>
-        </friction>
-        <bounce>
-          <restitution_coefficient>0</restitution_coefficient>
-          <threshold>0</threshold>
-        </bounce>
-        <contact>
-          <ode>
-            <soft_cfm>0</soft_cfm>
-            <soft_erp>0.200000</soft_erp>
-            <kp>10000000000000.000000</kp>
-            <kd>100000000000.000000</kd>
-            <max_vel>-1</max_vel>
-            <min_depth>0</min_depth>
-          </ode>
-        </contact>
-      </surface>
+      <gravity>true</gravity>
+      <maxVel>-1</maxVel>
+      <minDepth>0</minDepth>
+      <mu1>0.3</mu1>
+      <mu2>0.3</mu2>
+      <fdir1></fdir1>
+      <kp>1000000.0</kp>
+      <kd>10000.0</kd>
+      <selfCollide>true</selfCollide>
     </gazebo>
     <gazebo reference="${name}_link_4">
-      <turnGravityOff>false</turnGravityOff>
-      <surface>
-        <friction>
-          <ode>
-            <mu>0</mu>
-            <mu2>0</mu2>
-            <fdir1>0 0 0</fdir1>
-            <slip1>0</slip1>
-            <slip2>0</slip2>
-	  </ode>
-        </friction>
-        <bounce>
-          <restitution_coefficient>0</restitution_coefficient>
-          <threshold>0</threshold>
-        </bounce>
-        <contact>
-          <ode>
-            <soft_cfm>0</soft_cfm>
-            <soft_erp>0.200000</soft_erp>
-            <kp>10000000000000.000000</kp>
-            <kd>100000000000.000000</kd>
-            <max_vel>-1</max_vel>
-            <min_depth>0</min_depth>
-          </ode>
-        </contact>
-      </surface>
+      <gravity>true</gravity>
+      <maxVel>-1</maxVel>
+      <minDepth>0</minDepth>
+      <mu1>0.3</mu1>
+      <mu2>0.3</mu2>
+      <fdir1></fdir1>
+      <kp>1000000.0</kp>
+      <kd>10000.0</kd>
+      <selfCollide>true</selfCollide>
     </gazebo>
     <gazebo reference="${name}_link_5">
-      <turnGravityOff>false</turnGravityOff>
-      <surface>
-        <friction>
-          <ode>
-            <mu>0</mu>
-            <mu2>0</mu2>
-            <fdir1>0 0 0</fdir1>
-            <slip1>0</slip1>
-            <slip2>0</slip2>
-	  </ode>
-        </friction>
-        <bounce>
-          <restitution_coefficient>0</restitution_coefficient>
-          <threshold>0</threshold>
-        </bounce>
-        <contact>
-          <ode>
-            <soft_cfm>0</soft_cfm>
-            <soft_erp>0.200000</soft_erp>
-            <kp>10000000000000.000000</kp>
-            <kd>100000000000.000000</kd>
-            <max_vel>-1</max_vel>
-            <min_depth>0</min_depth>
-          </ode>
-        </contact>
-      </surface>
+      <gravity>true</gravity>
+      <maxVel>-1</maxVel>
+      <minDepth>0</minDepth>
+      <mu1>0.3</mu1>
+      <mu2>0.3</mu2>
+      <fdir1></fdir1>
+      <kp>1000000.0</kp>
+      <kd>10000.0</kd>
+      <selfCollide>true</selfCollide>
     </gazebo>
   </xacro:macro>

File: ahl_robot/youbot/virtual_youbot/ahl_youbot_description/urdf/arm/arm.urdf.xacro (robot description, xacro)
@@ -38,5 +38,5 @@
       <child link="${name}_link_1"/>
       <axis xyz="0 0 1"/>
-      <dynamics damping="0.1" friction="0"/>
+      <dynamics damping="0.7" friction="0"/>
       <limit effort="9.5" velocity="2.5" lower="${joint_1_lower_limit}" upper="${joint_1_upper_limit}"/>
     </joint>
@@ -65,5 +65,5 @@
       <child link="${name}_link_2"/>
       <axis xyz="0 1 0"/>
-      <dynamics damping="0.1" friction="0" />
+      <dynamics damping="0.7" friction="0" />
       <limit effort="9.5" velocity="2.5" lower="${joint_2_lower_limit}" upper="${joint_2_upper_limit}"/>
     </joint>
@@ -92,5 +92,5 @@
       <child link="${name}_link_3"/>
       <axis xyz="0 1 0"/>
-      <dynamics damping="0.1" friction="0"/>
+      <dynamics damping="0.7" friction="0"/>
       <limit effort="6.0" velocity="2.5" lower="${joint_3_lower_limit}" upper="${joint_3_upper_limit}"/>
     </joint>
@@ -119,5 +119,5 @@
       <child link="${name}_link_4"/>
       <axis xyz="0 1 0"/>
-      <dynamics damping="0.1" friction="0"/>
+      <dynamics damping="0.7" friction="0"/>
       <limit effort="2.0" velocity="1.5" lower="${joint_4_lower_limit}" upper="${joint_4_upper_limit}"/>
     </joint>
@@ -146,5 +146,5 @@
       <child link="${name}_link_5"/>
       <axis xyz="0 0 1"/>
-      <dynamics damping="0.1" friction="0"/>
+      <dynamics damping="0.7" friction="0"/>
       <limit effort="1.0" velocity="1.5" lower="${joint_5_lower_limit}" upper="${joint_5_upper_limit}"/>
     </joint>

Commit message: Deleted temporary files.

File: ahl_robot/youbot/virtual_youbot/ahl_youbot_description/urdf/arm/arm.gazebo.xacro (robot description, xacro)
@@ -9,10 +9,9 @@
       <maxVel>-1</maxVel>
       <minDepth>0</minDepth>
-      <mu1>0.3</mu1>
-      <mu2>0.3</mu2>
-      <fdir1></fdir1>
-      <kp>1000000.0</kp>
-      <kd>10000.0</kd>
-      <selfCollide>true</selfCollide>
+      <mu1>0</mu1>
+      <mu2>0</mu2>
+      <kp>10000000000.0</kp>
+      <kd>100000000.0</kd>
+      <selfCollide>false</selfCollide>
     </gazebo>
     <gazebo reference="${name}_link_1">
@@ -20,10 +19,9 @@
       <maxVel>-1</maxVel>
       <minDepth>0</minDepth>
-      <mu1>0.3</mu1>
-      <mu2>0.3</mu2>
-      <fdir1></fdir1>
-      <kp>1000000.0</kp>
-      <kd>10000.0</kd>
-      <selfCollide>true</selfCollide>
+      <mu1>0</mu1>
+      <mu2>0</mu2>
+      <kp>10000000000.0</kp>
+      <kd>100000000.0</kd>
+      <selfCollide>false</selfCollide>
     </gazebo>
     <gazebo reference="${name}_link_2">
@@ -31,10 +29,9 @@
       <maxVel>-1</maxVel>
       <minDepth>0</minDepth>
-      <mu1>0.3</mu1>
-      <mu2>0.3</mu2>
-      <fdir1></fdir1>
-      <kp>1000000.0</kp>
-      <kd>10000.0</kd>
-      <selfCollide>true</selfCollide>
+      <mu1>0</mu1>
+      <mu2>0</mu2>
+      <kp>10000000000.0</kp>
+      <kd>100000000.0</kd>
+      <selfCollide>false</selfCollide>
     </gazebo>
     <gazebo reference="${name}_link_3">
@@ -42,10 +39,9 @@
       <maxVel>-1</maxVel>
       <minDepth>0</minDepth>
-      <mu1>0.3</mu1>
-      <mu2>0.3</mu2>
-      <fdir1></fdir1>
-      <kp>1000000.0</kp>
-      <kd>10000.0</kd>
-      <selfCollide>true</selfCollide>
+      <mu1>0</mu1>
+      <mu2>0</mu2>
+      <kp>10000000000.0</kp>
+      <kd>100000000.0</kd>
+      <selfCollide>false</selfCollide>
     </gazebo>
     <gazebo reference="${name}_link_4">
@@ -53,10 +49,9 @@
       <maxVel>-1</maxVel>
       <minDepth>0</minDepth>
-      <mu1>0.3</mu1>
-      <mu2>0.3</mu2>
-      <fdir1></fdir1>
-      <kp>1000000.0</kp>
-      <kd>10000.0</kd>
-      <selfCollide>true</selfCollide>
+      <mu1>0</mu1>
+      <mu2>0</mu2>
+      <kp>10000000000.0</kp>
+      <kd>100000000.0</kd>
+      <selfCollide>false</selfCollide>
     </gazebo>
     <gazebo reference="${name}_link_5">
@@ -64,10 +59,9 @@
       <maxVel>-1</maxVel>
       <minDepth>0</minDepth>
-      <mu1>0.3</mu1>
-      <mu2>0.3</mu2>
-      <fdir1></fdir1>
-      <kp>1000000.0</kp>
-      <kd>10000.0</kd>
-      <selfCollide>true</selfCollide>
+      <mu1>0</mu1>
+      <mu2>0</mu2>
+      <kp>10000000000.0</kp>
+      <kd>100000000.0</kd>
+      <selfCollide>false</selfCollide>
     </gazebo>
   </xacro:macro>

File: ahl_robot/youbot/virtual_youbot/ahl_youbot_description/urdf/arm/arm.transmission.xacro (robot description, xacro)
@@ -6,5 +6,5 @@
   <!-- reduction ratio doesn't affect the model-->
   <!-- reduction ratio must not to be 0-->
-  <xacro:macro name="arm_transmission" params="name">
+  <xacro:macro name="youbot_arm_transmission" params="name">
     <transmission name="${name}_trans_1">
       <type>transmission_interface/SimpleTransmission</type>

File: ahl_robot/youbot/virtual_youbot/ahl_youbot_description/urdf/arm/arm.urdf.xacro (robot description, xacro)
@@ -38,5 +38,5 @@
       <child link="${name}_link_1"/>
       <axis xyz="0 0 1"/>
-      <dynamics damping="0.7" friction="0"/>
+      <dynamics damping="0.8" friction="0"/>
       <limit effort="9.5" velocity="2.5" lower="${joint_1_lower_limit}" upper="${joint_1_upper_limit}"/>
     </joint>
@@ -65,5 +65,5 @@
       <child link="${name}_link_2"/>
       <axis xyz="0 1 0"/>
-      <dynamics damping="0.7" friction="0" />
+      <dynamics damping="0.3" friction="0" />
       <limit effort="9.5" velocity="2.5" lower="${joint_2_lower_limit}" upper="${joint_2_upper_limit}"/>
     </joint>
@@ -92,5 +92,5 @@
       <child link="${name}_link_3"/>
       <axis xyz="0 1 0"/>
-      <dynamics damping="0.7" friction="0"/>
+      <dynamics damping="0.3" friction="0"/>
       <limit effort="6.0" velocity="2.5" lower="${joint_3_lower_limit}" upper="${joint_3_upper_limit}"/>
     </joint>
@@ -119,5 +119,5 @@
       <child link="${name}_link_4"/>
       <axis xyz="0 1 0"/>
-      <dynamics damping="0.7" friction="0"/>
+      <dynamics damping="0.3" friction="0"/>
       <limit effort="2.0" velocity="1.5" lower="${joint_4_lower_limit}" upper="${joint_4_upper_limit}"/>
     </joint>
@@ -146,5 +146,5 @@
       <child link="${name}_link_5"/>
       <axis xyz="0 0 1"/>
-      <dynamics damping="0.7" friction="0"/>
+      <dynamics damping="0.3" friction="0"/>
       <limit effort="1.0" velocity="1.5" lower="${joint_5_lower_limit}" upper="${joint_5_upper_limit}"/>
     </joint>

File: ahl_robot/youbot/virtual_youbot/ahl_youbot_description/urdf/base/base.gazebo.xacro (robot description, xacro)
@@ -9,10 +9,9 @@
       <maxVel>-1</maxVel>
       <minDepth>0</minDepth>
-      <mu1>0.5</mu1>
-      <mu2>0.5</mu2>
-      <fdir1></fdir1>
-      <kp>1000000.0</kp>
-      <kd>10000.0</kd>
-      <selfCollide>true</selfCollide>
+      <mu1>0</mu1>
+      <mu2>0</mu2>
+      <kp>10000000000.0</kp>
+      <kd>100000000.0</kd>
+      <selfCollide>0</selfCollide>
     </gazebo>
     <!-- front left wheel -->
@@ -21,10 +20,9 @@
       <maxVel>-1</maxVel>
       <minDepth>0</minDepth>
-      <mu1>1000.0</mu1>
-      <mu2>1000.0</mu2>
-      <fdir1></fdir1>
-      <kp>1000000.0</kp>
-      <kd>10000.0</kd>
-      <selfCollide>true</selfCollide>
+      <mu1>10000.0</mu1>
+      <mu2>10000.0</mu2>
+      <kp>10000000000.0</kp>
+      <kd>100000000.0</kd>
+      <selfCollide>0</selfCollide>
     </gazebo>
     <gazebo reference="caster_link_fl">
@@ -35,10 +33,9 @@
       <maxVel>-1</maxVel>
       <minDepth>0</minDepth>
-      <mu1>1000.0</mu1>
-      <mu2>1000.0</mu2>
-      <fdir1></fdir1>
-      <kp>1000000.0</kp>
-      <kd>10000.0</kd>
-      <selfCollide>true</selfCollide>
+      <mu1>10000.0</mu1>
+      <mu2>10000.0</mu2>
+      <kp>10000000000.0</kp>
+      <kd>100000000.0</kd>
+      <selfCollide>0</selfCollide>
     </gazebo>
     <gazebo reference="caster_link_fr">
@@ -49,10 +46,9 @@
       <maxVel>-1</maxVel>
       <minDepth>0</minDepth>
-      <mu1>1000.0</mu1>
-      <mu2>1000.0</mu2>
-      <fdir1></fdir1>
-      <kp>1000000.0</kp>
-      <kd>10000.0</kd>
-      <selfCollide>true</selfCollide>
+      <mu1>10000.0</mu1>
+      <mu2>10000.0</mu2>
+      <kp>10000000000.0</kp>
+      <kd>100000000.0</kd>
+      <selfCollide>0</selfCollide>
     </gazebo>
     <gazebo reference="caster_link_bl">
@@ -63,10 +59,9 @@
       <maxVel>-1</maxVel>
       <minDepth>0</minDepth>
-      <mu1>1000.0</mu1>
-      <mu2>1000.0</mu2>
-      <fdir1></fdir1>
+      <mu1>10000.0</mu1>
+      <mu2>10000.0</mu2>
       <kp>1000000.0</kp>
       <kd>10000.0</kd>
-      <selfCollide>true</selfCollide>
+      <selfCollide>0</selfCollide>
     </gazebo>
     <gazebo reference="caster_link_br">

File: ahl_robot/youbot/virtual_youbot/ahl_youbot_description/urdf/base/base.urdf.xacro (robot description, xacro)
@@ -69,12 +69,12 @@
     </link>
     <!-- front left wheel -->
-    <joint name="caster_joint_fl" type="fixed">
+    <joint name="caster_joint_fl" type="continuous">
       <origin xyz="${caster_offset_x} ${caster_offset_y} ${caster_offset_z}" rpy="0 0 0"/>
-      <axis xyz="0 1 0"/>
-      <limit effort="${caster_joint_effort}" velocity="${caster_joint_velocity}"/>
-      <dynamics damping="${caster_joint_damping}" friction="${caster_joint_friction}"/>
-      <safety_controller k_velocity="${caster_joint_safety_k_velocity}"/>
       <parent link="${name}_link"/>
       <child link="caster_link_fl"/>
+      <axis xyz="0 1 0"/>
+      <limit effort="${caster_joint_effort}" velocity="${caster_joint_velocity}"/>
+      <dynamics damping="${caster_joint_damping}" friction="${caster_joint_friction}"/>
+      <safety_controller k_velocity="${caster_joint_safety_k_velocity}"/>
     </joint>
     <link name="caster_link_fl">
@@ -114,12 +114,12 @@
     </link>
     <!-- front right wheel -->
-    <joint name="caster_joint_fr" type="fixed">
+    <joint name="caster_joint_fr" type="continuous">
       <origin xyz="${caster_offset_x} ${-caster_offset_y} ${caster_offset_z}" rpy="0 0 0"/>
-      <axis xyz="0 1 0"/>
-      <limit effort="${caster_joint_effort}" velocity="${caster_joint_velocity}"/>
-      <dynamics damping="${caster_joint_damping}" friction="${caster_joint_friction}"/>
-      <safety_controller k_velocity="${caster_joint_safety_k_velocity}"/>
       <parent link="${name}_link"/>
       <child link="caster_link_fr"/>
+      <axis xyz="0 1 0"/>
+      <limit effort="${caster_joint_effort}" velocity="${caster_joint_velocity}"/>
+      <dynamics damping="${caster_joint_damping}" friction="${caster_joint_friction}"/>
+      <safety_controller k_velocity="${caster_joint_safety_k_velocity}"/>
     </joint>
     <link name="caster_link_fr">
@@ -159,12 +159,12 @@
     </link>
     <!-- back left wheel -->
-    <joint name="caster_joint_bl" type="fixed">
+    <joint name="caster_joint_bl" type="continuous">
       <origin xyz="${-caster_offset_x} ${caster_offset_y} ${caster_offset_z}" rpy="0 0 0"/>
-      <axis xyz="0 1 0"/>
-      <limit effort="${caster_joint_effort}" velocity="${caster_joint_velocity}"/>
-      <dynamics damping="${caster_joint_damping}" friction="${caster_joint_friction}"/>
-      <safety_controller k_velocity="${caster_joint_safety_k_velocity}"/>
       <parent link="${name}_link"/>
       <child link="caster_link_bl"/>
+      <axis xyz="0 1 0"/>
+      <limit effort="${caster_joint_effort}" velocity="${caster_joint_velocity}"/>
+      <dynamics damping="${caster_joint_damping}" friction="${caster_joint_friction}"/>
+      <safety_controller k_velocity="${caster_joint_safety_k_velocity}"/>
     </joint>
     <link name="caster_link_bl">
@@ -204,12 +204,12 @@
     </link>
     <!-- back right wheel -->
-    <joint name="caster_joint_br" type="fixed">
+    <joint name="caster_joint_br" type="continuous">
       <origin xyz="${-caster_offset_x} ${-caster_offset_y} ${caster_offset_z}" rpy="0 0 0"/>
-      <axis xyz="0 1 0"/>
-      <limit effort="${caster_joint_effort}" velocity="${caster_joint_velocity}"/>
-      <dynamics damping="${caster_joint_damping}" friction="${caster_joint_friction}"/>
-      <safety_controller k_velocity="${caster_joint_safety_k_velocity}"/>
       <parent link="${name}_link"/>
       <child link="caster_link_br"/>
+      <axis xyz="0 1 0"/>
+      <limit effort="${caster_joint_effort}" velocity="${caster_joint_velocity}"/>
+      <dynamics damping="${caster_joint_damping}" friction="${caster_joint_friction}"/>
+      <safety_controller k_velocity="${caster_joint_safety_k_velocity}"/>
     </joint>
     <link name="caster_link_br">

File: ahl_robot/youbot/virtual_youbot/ahl_youbot_description/urdf/gripper/gripper.gazebo.xacro (robot description, xacro)
@@ -6,16 +6,31 @@
   <xacro:macro name="gripper_gazebo" params="name">
     <gazebo reference="${name}_palm_link">
-      <material>Gazebo/Black</material>
-      <turnGravityOff>false</turnGravityOff>
-      <selfCollide>true</selfCollide>
+      <gravity>true</gravity>
+      <maxVel>-1</maxVel>
+      <minDepth>0</minDepth>
+      <mu1>0</mu1>
+      <mu2>0</mu2>
+      <kp>10000000000.0</kp>
+      <kd>100000000.0</kd>
+      <selfCollide>false</selfCollide>
     </gazebo>
     <gazebo reference="${name}_finger_l_link">
-      <material>Gazebo/Black</material>
-      <turnGravityOff>false</turnGravityOff>
+      <gravity>true</gravity>
+      <maxVel>-1</maxVel>
+      <minDepth>0</minDepth>
+      <mu1>0.5</mu1>
+      <mu2>0</mu2>
+      <kp>10000000000.0</kp>
+      <kd>100000000.0</kd>
       <selfCollide>true</selfCollide>
     </gazebo>
     <gazebo reference="${name}_finger_r_link">
-      <material>Gazebo/Black</material>
-      <turnGravityOff>false</turnGravityOff>
+      <gravity>true</gravity>
+      <maxVel>-1</maxVel>
+      <minDepth>0</minDepth>
+      <mu1>0.5</mu1>
+      <mu2>0</mu2>
+      <kp>10000000000.0</kp>
+      <kd>100000000.0</kd>
       <selfCollide>true</selfCollide>
     </gazebo>

File: ahl_robot/youbot/virtual_youbot/ahl_youbot_description/urdf/gripper/gripper.urdf.xacro (robot description, xacro)
@@ -25,5 +25,4 @@
           <mesh filename="package://ahl_youbot_description/meshes/gripper/palm.dae"/>
         </geometry>
-        <material name="Black"/>
       </visual>
       <collision>
@@ -39,5 +38,5 @@
       <child link="${name}_finger_link_l"/>
       <axis xyz="0 1 0"/>
-      <dynamics damping="5.0" friction="0.5"/>
+      <dynamics damping="10.0" friction="0"/>
       <limit effort="0.5" velocity="0.1" lower="0" upper="${finger_joint}"/>
     </joint>
@@ -66,5 +65,5 @@
       <child link="${name}_finger_link_r"/>
       <axis xyz="0 1 0"/>
-      <dynamics damping="5.0" friction="0.5"/>
+      <dynamics damping="10.0" friction="0"/>
       <limit effort="0.5" velocity="0.1" lower="-${finger_joint}" upper="0"/>
     </joint>

File: ahl_robot/youbot/virtual_youbot/ahl_youbot_description/urdf/youbot.urdf.xacro (robot description, xacro)
@@ -8,7 +8,5 @@
   <xacro:include filename="$(find ahl_youbot_description)/urdf/arm/arm.urdf.xacro"/>
   <xacro:include filename="$(find ahl_youbot_description)/urdf/gripper/gripper.urdf.xacro"/>
-<!--
-  <xacro:include filename="$(find ahl_youbot_description)/controller/ros_controller.urdf.xacro"/>
--->
+<!--  <xacro:include filename="$(find ahl_youbot_description)/urdf/controller/ros_controller.urdf.xacro"/>-->
   <xacro:youbot_base    name="base"/>
   <xacro:youbot_arm     name="arm"/>
