Commit message: Created Mobility class for ahl_robot package. Now it can treat wheel-driven mobility.
Added 2 prismatic joints and 1 revolute joint to urdf of youbot. It simulates the motion of base.

Fixed some test codes.

File: ahl_robot/youbot/virtual_youbot/ahl_youbot_description/urdf/arm/arm.gazebo.xacro (robot description, xacro)
@@ -4,7 +4,7 @@
        xmlns:interface="http://playerstage.sourceforge.net/gazebo/xmlschema/#interface"
        xmlns:xacro="http://ros.org/wiki/xacro">
-  <xacro:macro name="arm_gazebo" params="name">
-    <gazebo reference="${name}_link_0">
-      <gravity>true</gravity>
+  <xacro:macro name="youbot_arm_gazebo" params="name">
+    <gazebo reference="link1">
+      <gravity>1</gravity>
       <maxVel>-1</maxVel>
       <minDepth>0</minDepth>
@@ -13,8 +13,8 @@
       <kp>10000000000.0</kp>
       <kd>100000000.0</kd>
-      <selfCollide>false</selfCollide>
+      <selfCollide>1</selfCollide>
     </gazebo>
-    <gazebo reference="${name}_link_1">
-      <gravity>true</gravity>
+    <gazebo reference="link2">
+      <gravity>1</gravity>
       <maxVel>-1</maxVel>
       <minDepth>0</minDepth>
@@ -23,8 +23,8 @@
       <kp>10000000000.0</kp>
       <kd>100000000.0</kd>
-      <selfCollide>false</selfCollide>
+      <selfCollide>1</selfCollide>
     </gazebo>
-    <gazebo reference="${name}_link_2">
-      <gravity>true</gravity>
+    <gazebo reference="link3">
+      <gravity>1</gravity>
       <maxVel>-1</maxVel>
       <minDepth>0</minDepth>
@@ -33,8 +33,8 @@
       <kp>10000000000.0</kp>
       <kd>100000000.0</kd>
-      <selfCollide>false</selfCollide>
+      <selfCollide>1</selfCollide>
     </gazebo>
-    <gazebo reference="${name}_link_3">
-      <gravity>true</gravity>
+    <gazebo reference="link4">
+      <gravity>1</gravity>
       <maxVel>-1</maxVel>
       <minDepth>0</minDepth>
@@ -43,8 +43,8 @@
       <kp>10000000000.0</kp>
       <kd>100000000.0</kd>
-      <selfCollide>false</selfCollide>
+      <selfCollide>1</selfCollide>
     </gazebo>
-    <gazebo reference="${name}_link_4">
-      <gravity>true</gravity>
+    <gazebo reference="link5">
+      <gravity>1</gravity>
       <maxVel>-1</maxVel>
       <minDepth>0</minDepth>
@@ -53,15 +53,5 @@
       <kp>10000000000.0</kp>
       <kd>100000000.0</kd>
-      <selfCollide>false</selfCollide>
-    </gazebo>
-    <gazebo reference="${name}_link_5">
-      <gravity>true</gravity>
-      <maxVel>-1</maxVel>
-      <minDepth>0</minDepth>
-      <mu1>0</mu1>
-      <mu2>0</mu2>
-      <kp>10000000000.0</kp>
-      <kd>100000000.0</kd>
-      <selfCollide>false</selfCollide>
+      <selfCollide>1</selfCollide>
     </gazebo>
   </xacro:macro>

File: ahl_robot/youbot/virtual_youbot/ahl_youbot_description/urdf/arm/arm.transmission.xacro (robot description, xacro)
@@ -13,5 +13,5 @@
         <mechanicalReduction>1</mechanicalReduction>
       </actuator>
-      <joint name="${name}_joint_1">
+      <joint name="joint1">
         <hardwareInterface>EffortJointInterface</hardwareInterface>
       </joint>
@@ -23,5 +23,5 @@
         <mechanicalReduction>1</mechanicalReduction>
       </actuator>
-      <joint name="${name}_joint_2">
+      <joint name="joint2">
         <hardwareInterface>EffortJointInterface</hardwareInterface>
       </joint>
@@ -33,5 +33,5 @@
         <mechanicalReduction>1</mechanicalReduction>
       </actuator>
-      <joint name="${name}_joint_3">
+      <joint name="joint3">
         <hardwareInterface>EffortJointInterface</hardwareInterface>
       </joint>
@@ -43,5 +43,5 @@
         <mechanicalReduction>1</mechanicalReduction>
       </actuator>
-      <joint name="${name}_joint_4">
+      <joint name="joint4">
         <hardwareInterface>EffortJointInterface</hardwareInterface>
       </joint>
@@ -53,5 +53,5 @@
         <mechanicalReduction>1</mechanicalReduction>
       </actuator>
-      <joint name="${name}_joint_5">
+      <joint name="joint5">
         <hardwareInterface>EffortJointInterface</hardwareInterface>
       </joint>

File: ahl_robot/youbot/virtual_youbot/ahl_youbot_description/urdf/base/base.gazebo.xacro (robot description, xacro)
@@ -5,6 +5,36 @@
        xmlns:xacro="http://ros.org/wiki/xacro">
   <xacro:macro name="youbot_base_gazebo">
+    <gazebo reference="base_x">
+      <gravity>0</gravity>
+      <maxVel>-1</maxVel>
+      <minDepth>0</minDepth>
+      <mu1>0</mu1>
+      <mu2>0</mu2>
+      <kp>10000000000.0</kp>
+      <kd>100000000.0</kd>
+      <selfCollide>0</selfCollide>
+    </gazebo>
+    <gazebo reference="base_y">
+      <gravity>0</gravity>
+      <maxVel>-1</maxVel>
+      <minDepth>0</minDepth>
+      <mu1>0</mu1>
+      <mu2>0</mu2>
+      <kp>10000000000.0</kp>
+      <kd>100000000.0</kd>
+      <selfCollide>0</selfCollide>
+    </gazebo>
+    <gazebo reference="base_yaw">
+      <gravity>0</gravity>
+      <maxVel>-1</maxVel>
+      <minDepth>0</minDepth>
+      <mu1>0</mu1>
+      <mu2>0</mu2>
+      <kp>10000000000.0</kp>
+      <kd>100000000.0</kd>
+      <selfCollide>0</selfCollide>
+    </gazebo>
     <gazebo reference="base_link">
-      <gravity>true</gravity>
+      <gravity>1</gravity>
       <maxVel>-1</maxVel>
       <minDepth>0</minDepth>
@@ -17,64 +47,58 @@
     <!-- front left wheel -->
     <gazebo reference="wheel_link_fl">
-      <gravity>true</gravity>
+      <gravity>1</gravity>
       <maxVel>-1</maxVel>
       <minDepth>0</minDepth>
-      <mu1>10000.0</mu1>
-      <mu2>10000.0</mu2>
+      <mu1>0</mu1>
+      <mu2>0</mu2>
       <kp>10000000000.0</kp>
       <kd>100000000.0</kd>
       <selfCollide>0</selfCollide>
     </gazebo>
-    <gazebo reference="caster_link_fl">
-    </gazebo>
     <!-- front right wheel -->
     <gazebo reference="wheel_link_fr">
-      <gravity>true</gravity>
+      <gravity>1</gravity>
       <maxVel>-1</maxVel>
       <minDepth>0</minDepth>
-      <mu1>10000.0</mu1>
-      <mu2>10000.0</mu2>
+      <mu1>0</mu1>
+      <mu2>0</mu2>
       <kp>10000000000.0</kp>
       <kd>100000000.0</kd>
       <selfCollide>0</selfCollide>
     </gazebo>
-    <gazebo reference="caster_link_fr">
-    </gazebo>
     <!-- back left wheel -->
     <gazebo reference="wheel_link_bl">
-      <gravity>true</gravity>
+      <gravity>1</gravity>
       <maxVel>-1</maxVel>
       <minDepth>0</minDepth>
-      <mu1>10000.0</mu1>
-      <mu2>10000.0</mu2>
+      <mu1>0</mu1>
+      <mu2>0</mu2>
       <kp>10000000000.0</kp>
       <kd>100000000.0</kd>
       <selfCollide>0</selfCollide>
     </gazebo>
-    <gazebo reference="caster_link_bl">
-    </gazebo>
     <!-- back right wheel -->
     <gazebo reference="wheel_link_br">
-      <gravity>true</gravity>
+      <gravity>1</gravity>
       <maxVel>-1</maxVel>
       <minDepth>0</minDepth>
-      <mu1>10000.0</mu1>
-      <mu2>10000.0</mu2>
+      <mu1>0</mu1>
+      <mu2>0</mu2>
       <kp>1000000.0</kp>
       <kd>10000.0</kd>
       <selfCollide>0</selfCollide>
     </gazebo>
-    <gazebo reference="caster_link_br">
-    </gazebo>
     <!-- position controller -->
+<!--
     <gazebo>
-<!--      <plugin name="base_controller" filename="libgazebo_ros_planar_move.so">
-        <commandTopic>cmd_vel</commandTopic>
+      <plugin name="base_controller" filename="libgazebo_ros_planar_move.so">
+        <commandTopic>youbot/cmd_vel</commandTopic>
         <odometryTopic>odom</odometryTopic>
         <odometryFrame>odom</odometryFrame>
-        <odometryRate>100.0</odometryRate>
-        <robotBaseFrame>base_footprint</robotBaseFrame>
-      </plugin>-->
+        <odometryRate>10.0</odometryRate>
+        <robotBaseFrame>base_link</robotBaseFrame>
+      </plugin>
     </gazebo>
+-->
   </xacro:macro>
 </robot>

File: ahl_robot/youbot/virtual_youbot/ahl_youbot_description/urdf/base/base.transmission.xacro (robot description, xacro)
@@ -4,89 +4,75 @@
        xmlns:interface="http://playerstage.sourceforge.net/gazebo/xmlschema/#interface"
        xmlns:xacro="http://ros.org/wiki/xacro">
-  <property name="wheel_mechanical_reduction" value="${624/35 * 80/18}"/>
-  <property name="caster_mechanical_reduction" value="${624/35 * 80/18}"/>
+<!--  <property name="wheel_mechanical_reduction" value="${624/35 * 80/18}"/> -->
+  <property name="wheel_mechanical_reduction" value="1"/>
   <xacro:macro name="youbot_base_transmission">
-  <!-- front left wheel -->
+    <transmission name="base_x_trans">
+      <type>transmission_interface/SimpleTransmission</type>
+      <actuator name="base_x_motor">
+        <hardwareInterface>EffortJointInterface</hardwareInterface>
+        <mechanicalReduction>1</mechanicalReduction>
+      </actuator>
+      <joint name="base_x_joint">
+        <hardwareInterface>EffortJointInterface</hardwareInterface>
+      </joint>
+    </transmission>
+    <transmission name="base_y_trans">
+      <type>transmission_interface/SimpleTransmission</type>
+      <actuator name="base_y_motor">
+        <hardwareInterface>EffortJointInterface</hardwareInterface>
+        <mechanicalReduction>1</mechanicalReduction>
+      </actuator>
+      <joint name="base_y_joint">
+        <hardwareInterface>EffortJointInterface</hardwareInterface>
+      </joint>
+    </transmission>
+    <transmission name="base_yaw_trans">
+      <type>transmission_interface/SimpleTransmission</type>
+      <actuator name="base_yaw_motor">
+        <hardwareInterface>EffortJointInterface</hardwareInterface>
+        <mechanicalReduction>1</mechanicalReduction>
+      </actuator>
+      <joint name="base_yaw_joint">
+        <hardwareInterface>EffortJointInterface</hardwareInterface>
+      </joint>
+    </transmission>
     <transmission name="wheel_trans_fl">
       <type>transmission_interface/SimpleTransmission</type>
       <actuator name="wheel_motor_fl">
-        <hardwareInterface>VelocityJointInterface</hardwareInterface>
+        <hardwareInterface>EffortJointInterface</hardwareInterface>
         <mechanicalReduction>${wheel_mechanical_reduction}</mechanicalReduction>
       </actuator>
       <joint name="wheel_joint_fl">
-        <hardwareInterface>VelocityJointInterface</hardwareInterface>
+        <hardwareInterface>EffortJointInterface</hardwareInterface>
       </joint>
     </transmission>
-    <transmission name="caster_trans_fl">
-      <type>transmission_interface/SimpleTransmission</type>
-       <actuator name="caster_motor_fl">
-        <hardwareInterface>VelocityJointInterface</hardwareInterface>
-        <mechanicalReduction>${caster_mechanical_reduction}</mechanicalReduction>
-      </actuator>
-      <joint name="caster_joint_fl">
-        <hardwareInterface>VelocityJointInterface</hardwareInterface>
-      </joint>
-    </transmission>
-    <!-- front right wheel -->
     <transmission name="wheel_trans_fr">
       <type>transmission_interface/SimpleTransmission</type>
       <actuator name="wheel_motor_fr">
-        <hardwareInterface>VelocityJointInterface</hardwareInterface>
+        <hardwareInterface>EffortJointInterface</hardwareInterface>
         <mechanicalReduction>${wheel_mechanical_reduction}</mechanicalReduction>
       </actuator>
       <joint name="wheel_joint_fr">
-        <hardwareInterface>VelocityJointInterface</hardwareInterface>
+        <hardwareInterface>EffortJointInterface</hardwareInterface>
       </joint>
     </transmission>
-    <transmission name="caster_trans_fr">
-      <type>transmission_interface/SimpleTransmission</type>
-      <actuator name="caster_motor_fr" >
-        <hardwareInterface>VelocityJointInterface</hardwareInterface>
-        <mechanicalReduction>${caster_mechanical_reduction}</mechanicalReduction>
-      </actuator>
-      <joint name="caster_joint_fr">
-        <hardwareInterface>VelocityJointInterface</hardwareInterface>
-      </joint>
-    </transmission>
-    <!-- back left wheel -->
     <transmission name="wheel_trans_bl">
       <type>transmission_interface/SimpleTransmission</type>
       <actuator name="wheel_motor_bl" >
-        <hardwareInterface>VelocityJointInterface</hardwareInterface>
+        <hardwareInterface>EffortJointInterface</hardwareInterface>
         <mechanicalReduction>${wheel_mechanical_reduction}</mechanicalReduction>
       </actuator>
       <joint name="wheel_joint_bl">
-        <hardwareInterface>VelocityJointInterface</hardwareInterface>
+        <hardwareInterface>EffortJointInterface</hardwareInterface>
       </joint>
     </transmission>
-    <transmission name="caster_trans_bl">
-      <type>transmission_interface/SimpleTransmission</type>
-      <actuator name="caster_motor_bl" >
-        <hardwareInterface>VelocityJointInterface</hardwareInterface>
-        <mechanicalReduction>${caster_mechanical_reduction}</mechanicalReduction>
-      </actuator>
-      <joint name="caster_joint_bl">
-        <hardwareInterface>VelocityJointInterface</hardwareInterface>
-      </joint>
-    </transmission>
-    <!-- back right wheel -->
     <transmission name="wheel_trans_br">
       <type>transmission_interface/SimpleTransmission</type>
       <actuator name="wheel_motor_br" >
-        <hardwareInterface>VelocityJointInterface</hardwareInterface>
+        <hardwareInterface>EffortJointInterface</hardwareInterface>
         <mechanicalReduction>${wheel_mechanical_reduction}</mechanicalReduction>
       </actuator>
       <joint name="wheel_joint_br">
-        <hardwareInterface>VelocityJointInterface</hardwareInterface>
-      </joint>
-    </transmission>
-    <transmission name="caster_trans_br">
-      <type>transmission_interface/SimpleTransmission</type>
-      <actuator name="caster_motor_br" >
-        <hardwareInterface>VelocityJointInterface</hardwareInterface>
-        <mechanicalReduction>${caster_mechanical_reduction}</mechanicalReduction>
-      </actuator>
-      <joint name="caster_joint_br">
-        <hardwareInterface>VelocityJointInterface</hardwareInterface>
+        <hardwareInterface>EffortJointInterface</hardwareInterface>
       </joint>
     </transmission>

File: ahl_robot/youbot/virtual_youbot/ahl_youbot_description/urdf/gripper/gripper.gazebo.xacro (robot description, xacro)
@@ -4,17 +4,7 @@
        xmlns:interface="http://playerstage.sourceforge.net/gazebo/xmlschema/#interface"
        xmlns:xacro="http://ros.org/wiki/xacro">
-  <xacro:macro name="gripper_gazebo" params="name">
-    <gazebo reference="${name}_palm_link">
-      <gravity>true</gravity>
-      <maxVel>-1</maxVel>
-      <minDepth>0</minDepth>
-      <mu1>0</mu1>
-      <mu2>0</mu2>
-      <kp>10000000000.0</kp>
-      <kd>100000000.0</kd>
-      <selfCollide>false</selfCollide>
-    </gazebo>
-    <gazebo reference="${name}_finger_l_link">
-      <gravity>true</gravity>
+  <xacro:macro name="youbot_gripper_gazebo" params="name">
+    <gazebo reference="finger_link_l">
+      <gravity>1</gravity>
       <maxVel>-1</maxVel>
       <minDepth>0</minDepth>
@@ -23,8 +13,8 @@
       <kp>10000000000.0</kp>
       <kd>100000000.0</kd>
-      <selfCollide>true</selfCollide>
+      <selfCollide>1</selfCollide>
     </gazebo>
-    <gazebo reference="${name}_finger_r_link">
-      <gravity>true</gravity>
+    <gazebo reference="finger_link_r">
+      <gravity>1</gravity>
       <maxVel>-1</maxVel>
       <minDepth>0</minDepth>
@@ -33,5 +23,5 @@
       <kp>10000000000.0</kp>
       <kd>100000000.0</kd>
-      <selfCollide>true</selfCollide>
+      <selfCollide>1</selfCollide>
     </gazebo>
   </xacro:macro>

File: ahl_robot/youbot/virtual_youbot/ahl_youbot_description/urdf/gripper/gripper.transmission.xacro (robot description, xacro)
@@ -5,21 +5,21 @@
        xmlns:xacro="http://ros.org/wiki/xacro">
   <xacro:macro name="youbot_gripper_transmission" params="name">
-    <transmission name="${name}_finger_l_trans">
+    <transmission name="finger_trans_l">
       <type>transmission_interface/SimpleTransmission</type>
-      <actuator name="${name}_finger_l_motor">
+      <actuator name="finger_motor_l">
         <hardwareInterface>EffortJointInterface</hardwareInterface>
         <mechanicalReduction>1</mechanicalReduction>
       </actuator>
-      <joint name="${name}_finger_joint_l">
+      <joint name="finger_joint_l">
         <hardwareInterface>EffortJointInterface</hardwareInterface>
       </joint>
     </transmission>
-    <transmission name="${name}_finger_r_trans">
+    <transmission name="finger_trans_r">
       <type>transmission_interface/SimpleTransmission</type>
-      <actuator name="${name}_finger_r_motor">
+      <actuator name="finger_motor_r">
         <hardwareInterface>EffortJointInterface</hardwareInterface>
         <mechanicalReduction>1</mechanicalReduction>
       </actuator>
-      <joint name="${name}_finger_joint_r">
+      <joint name="finger_joint_r">
         <hardwareInterface>EffortJointInterface</hardwareInterface>
       </joint>
