Commit message: Modified physical parameters, such as damping, mass, self_collide flag and so on. Especially, damping of finger_tip is very important. It should be small, because it has very small mass and damping is unstable.

File: ahl_robot/ahl_pr2_description/urdf/arm/arm.gazebo.xacro (robot description, xacro)
@@ -24,5 +24,5 @@
       <kp>10000000000.0</kp>
       <kd>100000000.0</kd>
-      <selfCollide>1</selfCollide>
+      <selfCollide>0</selfCollide>
     </gazebo>
     <gazebo reference="upper_arm_l_link">
@@ -74,5 +74,5 @@
       <kp>10000000000.0</kp>
       <kd>100000000.0</kd>
-      <selfCollide>0</selfCollide>
+      <selfCollide>1</selfCollide>
     </gazebo>
     <!-- right arm -->
@@ -95,5 +95,5 @@
       <kp>10000000000.0</kp>
       <kd>100000000.0</kd>
-      <selfCollide>1</selfCollide>
+      <selfCollide>0</selfCollide>
     </gazebo>
     <gazebo reference="upper_arm_r_link">
@@ -145,5 +145,5 @@
       <kp>10000000000.0</kp>
       <kd>100000000.0</kd>
-      <selfCollide>0</selfCollide>
+      <selfCollide>1</selfCollide>
     </gazebo>
   </xacro:macro>

File: ahl_robot/ahl_pr2_description/urdf/base/base.gazebo.xacro (robot description, xacro)
@@ -43,5 +43,5 @@
       <kp>10000000000.0</kp>
       <kd>100000000.0</kd>
-      <selfCollide>1</selfCollide>
+      <selfCollide>0</selfCollide>
     </gazebo>
     <gazebo reference="caster_fl_link">
@@ -133,5 +133,5 @@
       <kp>10000000000.0</kp>
       <kd>100000000.0</kd>
-      <selfCollide>1</selfCollide>
+      <selfCollide>0</selfCollide>
     </gazebo>
   </xacro:macro>

File: ahl_robot/ahl_pr2_description/urdf/base/base.property.xacro (robot description, xacro)
@@ -67,5 +67,5 @@
   <xacro:macro name="base_link_inertial">
     <inertial>
-      <mass value="118"/>
+      <mass value="118.0"/>
       <origin xyz="-0.062 0 0.201"/>
       <inertia ixx="8.431730" ixy="0" ixz="0" iyy="8.533050" iyz="0" izz="3.787470"/>
@@ -93,5 +93,5 @@
     </visual>
   </xacro:macro>
-  <property name="caster_damping" value="1"/>
+  <property name="caster_damping" value="0.7"/>
   <property name="caster_friction" value="0.2"/>
   <property name="caster_effort" value="10000"/>
@@ -109,5 +109,5 @@
   <property name="wheel_radius" value="0.075"/>
   <property name="wheel_length" value="0.10"/>
-  <property name="wheel_damping" value="1"/>
+  <property name="wheel_damping" value="0.7"/>
   <property name="wheel_friction" value="0.2"/>
   <property name="wheel_effort" value="10000"/>

File: ahl_robot/ahl_pr2_description/urdf/gripper/gripper.property.xacro (robot description, xacro)
@@ -12,8 +12,8 @@
     </inertial>
   </xacro:macro>
-  <property name="finger_damping" value="1"/>
-  <property name="finger_friction" value="1"/>
+  <property name="finger_damping" value="0.2"/>
+  <property name="finger_friction" value="0.7"/>
   <property name="finger_effort" value="10000"/>
-  <property name="finger_velocity" value="10000"/>
+  <property name="finger_velocity" value="0.1"/>
   <property name="finger_upper" value="0.548"/>
   <property name="finger_lower" value="0"/>
@@ -23,13 +23,13 @@
   <xacro:macro name="finger_tip_inertial">
     <inertial>
-      <mass value="0.4419"/>
+      <mass value="0.04419"/>
       <origin xyz="0.004 0 0" rpy="0 0 0"/>
-      <inertia ixx="0.0001" ixy="0" ixz="0" iyy="0.0001" iyz="0" izz="0.0001"/>
+      <inertia ixx="0.00001" ixy="0" ixz="0" iyy="0.00001" iyz="0" izz="0.00001"/>
     </inertial>
   </xacro:macro>
-  <property name="finger_tip_damping" value="1"/>
-  <property name="finger_tip_friction" value="1"/>
+  <property name="finger_tip_damping" value="0.2"/>
+  <property name="finger_tip_friction" value="0.7"/>
   <property name="finger_tip_effort" value="10000"/>
-  <property name="finger_tip_velocity" value="10000"/>
+  <property name="finger_tip_velocity" value="0.1"/>
   <property name="finger_tip_upper" value="0.548"/>
   <property name="finger_tip_lower" value="0"/>
