Commit message: Modified wrist_roll_link and deleted gripper_palm_link.
Modified physical parameters.

Now I can use this model for experiment.

File: ahl_robot/ahl_pr2_description/urdf/arm/arm.property.xacro (robot description, xacro)
@@ -7,15 +7,15 @@
   <xacro:macro name="shoulder_pan_inertial">
     <inertial>
-      <mass value="3"/>
-      <origin xyz="0 0 0" rpy="0 0 0"/>
-      <inertia ixx="0.1" ixy="0" ixz="0" iyy="0.1" iyz="0" izz="0.1"/>
+      <mass value="25.799"/>
+      <origin xyz="-0.001 0 -0.098" rpy="0 0 0"/>
+      <inertia ixx="0.866179" ixy="0" ixz="0" iyy="0.874217" iyz="0" izz="0.273538"/>
     </inertial>
   </xacro:macro>
-  <property name="shoulder_pan_damping" value="1"/>
+  <property name="shoulder_pan_damping" value="0.7"/>
   <property name="shoulder_pan_friction" value="0"/>
   <property name="shoulder_pan_effort" value="10000"/>
   <property name="shoulder_pan_velocity" value="10000"/>
-  <property name="shoulder_pan_upper" value="${M_PI / 2}"/>
-  <property name="shoulder_pan_lower" value="${-M_PI / 2}"/>
+  <property name="shoulder_pan_upper" value="2.285404"/>
+  <property name="shoulder_pan_lower" value="-0.714602"/>
   <property name="shoulder_lift_x" value="0.1"/>
   <property name="shoulder_lift_y" value="0"/>
@@ -23,15 +23,15 @@
   <xacro:macro name="shoulder_lift_inertial">
     <inertial>
-      <mass value="3"/>
-      <origin xyz="0 0 0" rpy="0 0 0"/>
-      <inertia ixx="0.1" ixy="0" ixz="0" iyy="0.1" iyz="0" izz="0.1"/>
+      <mass value="2.750"/>
+      <origin xyz="0.02195 0 -0.03127" rpy="0 0 0"/>
+      <inertia ixx="0.021056" ixy="0" ixz="0" iyy="0.021272" iyz="0" izz="0.019758"/>
     </inertial>
   </xacro:macro>
-  <property name="shoulder_lift_damping" value="1"/>
+  <property name="shoulder_lift_damping" value="0.7"/>
   <property name="shoulder_lift_friction" value="0"/>
   <property name="shoulder_lift_effort" value="10000"/>
   <property name="shoulder_lift_velocity" value="10000"/>
-  <property name="shoulder_lift_upper" value="${M_PI / 2}"/>
-  <property name="shoulder_lift_lower" value="${-M_PI / 2}"/>
+  <property name="shoulder_lift_upper" value="1.396300"/>
+  <property name="shoulder_lift_lower" value="-0.523601"/>
   <property name="upper_arm_x" value="0.12"/>
   <property name="upper_arm_y" value="0"/>
@@ -39,15 +39,15 @@
   <xacro:macro name="upper_arm_inertial">
     <inertial>
-      <mass value="3"/>
-      <origin xyz="0 0 0" rpy="0 0 0"/>
-      <inertia ixx="0.1" ixy="0" ixz="0" iyy="0.1" iyz="0" izz="0.1"/>
+      <mass value="6.118"/>
+      <origin xyz="0.211 0 -0.001" rpy="0 0 0"/>
+      <inertia ixx="0.025306" ixy="0" ixz="0" iyy="0.084737" iyz="0" izz="0.086016"/>
     </inertial>
   </xacro:macro>
-  <property name="upper_arm_damping" value="1"/>
+  <property name="upper_arm_damping" value="0.4"/>
   <property name="upper_arm_friction" value="0"/>
   <property name="upper_arm_effort" value="10000"/>
   <property name="upper_arm_velocity" value="10000"/>
-  <property name="upper_arm_upper" value="${M_PI / 2}"/>
-  <property name="upper_arm_lower" value="${-M_PI / 2}"/>
+  <property name="upper_arm_upper" value="3.900008"/>
+  <property name="upper_arm_lower" value="-0.800000"/>
   <property name="elbow_x" value="0.28"/>
   <property name="elbow_y" value="0"/>
@@ -55,15 +55,15 @@
   <xacro:macro name="elbow_inertial">
     <inertial>
-      <mass value="3"/>
-      <origin xyz="0 0 0" rpy="0 0 0"/>
-      <inertia ixx="0.1" ixy="0" ixz="0" iyy="0.1" iyz="0" izz="0.1"/>
+      <mass value="1.903"/>
+      <origin xyz="0.010 0 -0.012" rpy="0 0 0"/>
+      <inertia ixx="0.003465" ixy="0" ixz="0" iyy="0.004416" iyz="0" izz="0.003592"/>
     </inertial>
   </xacro:macro>
-  <property name="elbow_damping" value="1"/>
+  <property name="elbow_damping" value="0.7"/>
   <property name="elbow_friction" value="0"/>
   <property name="elbow_effort" value="10000"/>
   <property name="elbow_velocity" value="10000"/>
-  <property name="elbow_upper" value="${M_PI / 2}"/>
-  <property name="elbow_lower" value="${-M_PI / 2}"/>
+  <property name="elbow_upper" value="0"/>
+  <property name="elbow_lower" value="-2.321305"/>
   <property name="forearm_x" value="0.09"/>
   <property name="forearm_y" value="0"/>
@@ -71,15 +71,15 @@
   <xacro:macro name="forearm_inertial">
     <inertial>
-      <mass value="3"/>
-      <origin xyz="0 0 0" rpy="0 0 0"/>
-      <inertia ixx="0.1" ixy="0" ixz="0" iyy="0.1" iyz="0" izz="0.1"/>
+      <mass value="2.690"/>
+      <origin xyz="0.181 0 -0.009" rpy="0 0 0"/>
+      <inertia ixx="0.014668" ixy="0" ixz="0" iyy="0.026279" iyz="0" izz="0.027775"/>
     </inertial>
   </xacro:macro>
-  <property name="forearm_damping" value="1"/>
+  <property name="forearm_damping" value="0.4"/>
   <property name="forearm_friction" value="0"/>
   <property name="forearm_effort" value="10000"/>
   <property name="forearm_velocity" value="10000"/>
-  <property name="forearm_upper" value="${M_PI / 2}"/>
-  <property name="forearm_lower" value="${-M_PI / 2}"/>
+  <property name="forearm_upper" value="10000000"/>
+  <property name="forearm_lower" value="-10000000"/>
   <property name="wrist_flex_x" value="0.23"/>
   <property name="wrist_flex_y" value="0"/>
@@ -87,15 +87,15 @@
   <xacro:macro name="wrist_flex_inertial">
     <inertial>
-      <mass value="3"/>
-      <origin xyz="0 0 0" rpy="0 0 0"/>
-      <inertia ixx="0.1" ixy="0" ixz="0" iyy="0.1" iyz="0" izz="0.1"/>
+      <mass value="0.614"/>
+      <origin xyz="-0.002 0 -0.001" rpy="0 0 0"/>
+      <inertia ixx="0.000652" ixy="0" ixz="0" iyy="0.000198" iyz="0" izz="0.000645"/>
     </inertial>
   </xacro:macro>
-  <property name="wrist_flex_damping" value="1"/>
+  <property name="wrist_flex_damping" value="0.4"/>
   <property name="wrist_flex_friction" value="0"/>
   <property name="wrist_flex_effort" value="10000"/>
   <property name="wrist_flex_velocity" value="10000"/>
-  <property name="wrist_flex_upper" value="${M_PI / 2}"/>
-  <property name="wrist_flex_lower" value="${-M_PI / 2}"/>
+  <property name="wrist_flex_upper" value="-2.180004"/>
+  <property name="wrist_flex_lower" value="0"/>
   <property name="wrist_roll_x" value="0.03"/>
   <property name="wrist_roll_y" value="0"/>
@@ -103,14 +103,14 @@
   <xacro:macro name="wrist_roll_inertial">
     <inertial>
-      <mass value="3"/>
-      <origin xyz="0 0 0" rpy="0 0 0"/>
-      <inertia ixx="0.1" ixy="0" ixz="0" iyy="0.1" iyz="0" izz="0.1"/>
+      <mass value="0.681"/>
+      <origin xyz="0.056 0 -0.001" rpy="0 0 0"/>
+      <inertia ixx="0.011352" ixy="0" ixz="0" iyy="0.011677" iyz="0" izz="0.011866"/>
     </inertial>
   </xacro:macro>
-  <property name="wrist_roll_damping" value="1"/>
+  <property name="wrist_roll_damping" value="0.4"/>
   <property name="wrist_roll_friction" value="0"/>
   <property name="wrist_roll_effort" value="10000"/>
   <property name="wrist_roll_velocity" value="10000"/>
-  <property name="wrist_roll_upper" value="${M_PI / 2}"/>
-  <property name="wrist_roll_lower" value="${-M_PI / 2}"/>
+  <property name="wrist_roll_upper" value="10000000"/>
+  <property name="wrist_roll_lower" value="-10000000"/>
 </robot>

File: ahl_robot/ahl_pr2_description/urdf/base/base.property.xacro (robot description, xacro)
@@ -4,5 +4,5 @@
   <xacro:macro name="base_x_inertial">
     <inertial>
-      <mass value="0.01"/>
+      <mass value="0.1"/>
       <origin xyz="0 0 0" rpy="0 0 0"/>
       <inertia ixx="100" ixy="0" ixz="0" iyy="100" iyz="0" izz="100"/>
@@ -18,5 +18,5 @@
   </xacro:macro>
   <property name="base_x_damping" value="3"/>
-  <property name="base_x_friction" value="0"/>
+  <property name="base_x_friction" value="0.2"/>
   <property name="base_x_effort" value="10000"/>
   <property name="base_x_velocity" value="10000"/>
@@ -25,5 +25,5 @@
   <xacro:macro name="base_y_inertial">
     <inertial>
-      <mass value="0.01"/>
+      <mass value="0.1"/>
       <origin xyz="0 0 0" rpy="0 0 0"/>
       <inertia ixx="100" ixy="0" ixz="0" iyy="100" iyz="0" izz="100"/>
@@ -39,5 +39,5 @@
   </xacro:macro>
   <property name="base_y_damping" value="3"/>
-  <property name="base_y_friction" value="0"/>
+  <property name="base_y_friction" value="0.2"/>
   <property name="base_y_effort" value="10000"/>
   <property name="base_y_velocity" value="10000"/>
@@ -46,5 +46,5 @@
   <xacro:macro name="base_yaw_inertial">
     <inertial>
-      <mass value="100"/>
+      <mass value="300"/>
       <origin xyz="0 0 0" rpy="0 0 0"/>
       <inertia ixx="0.001" ixy="0" ixz="0" iyy="0.001" iyz="0" izz="0.001"/>
@@ -60,5 +60,5 @@
   </xacro:macro>
   <property name="base_yaw_damping" value="3"/>
-  <property name="base_yaw_friction" value="0"/>
+  <property name="base_yaw_friction" value="0.2"/>
   <property name="base_yaw_effort" value="10000"/>
   <property name="base_yaw_velocity" value="10000"/>
@@ -67,7 +67,7 @@
   <xacro:macro name="base_link_inertial">
     <inertial>
-      <mass value="100"/>
-      <origin xyz="0 0 0"/>
-      <inertia ixx="1" ixy="0" ixz="0" iyy="1" iyz="0" izz="1"/>
+      <mass value="118"/>
+      <origin xyz="-0.062 0 0.201"/>
+      <inertia ixx="8.431730" ixy="0" ixz="0" iyy="8.533050" iyz="0" izz="3.787470"/>
     </inertial>
   </xacro:macro>
@@ -77,7 +77,7 @@
   <xacro:macro name="caster_inertial">
     <inertial>
-      <mass value="1"/>
+      <mass value="3.47"/>
       <origin xyz="0 0 0" rpy="0 0 0"/>
-      <inertia ixx="0.01" ixy="0" ixz="0" iyy="0.01" iyz="0" izz="0.01"/>
+      <inertia ixx="0.012412" ixy="0" ixz="0" iyy="0.015218" iyz="0" izz="0.011764"/>
     </inertial>
   </xacro:macro>
@@ -88,8 +88,11 @@
         <box size="0.12 0.02 0.2"/>
       </geometry>
+      <material name="caster_gray">
+        <color rgba="0.4 0.4 0.4 1"/>
+      </material>
     </visual>
   </xacro:macro>
   <property name="caster_damping" value="1"/>
-  <property name="caster_friction" value="0"/>
+  <property name="caster_friction" value="0.2"/>
   <property name="caster_effort" value="10000"/>
   <property name="caster_velocity" value="10000"/>
@@ -99,7 +102,7 @@
   <xacro:macro name="wheel_inertial">
     <inertial>
-      <mass value="2"/>
+      <mass value="0.880"/>
       <origin xyz="0 0 0" rpy="0 0 0"/>
-      <inertia ixx="0.01" ixy="0" ixz="0" iyy="0.01" iyz="0" izz="0.01"/>
+      <inertia ixx="0.012412" ixy="0" ixz="0" iyy="0.015218" iyz="0" izz="0.011764"/>
     </inertial>
   </xacro:macro>
@@ -107,5 +110,5 @@
   <property name="wheel_length" value="0.10"/>
   <property name="wheel_damping" value="1"/>
-  <property name="wheel_friction" value="0"/>
+  <property name="wheel_friction" value="0.2"/>
   <property name="wheel_effort" value="10000"/>
   <property name="wheel_velocity" value="10000"/>
@@ -117,14 +120,14 @@
   <xacro:macro name="torso_inertial">
     <inertial>
-      <mass value="20"/>
-      <origin xyz="0 0 0" rpy="0 0 0"/>
-      <inertia ixx="0.1" ixy="0" ixz="0" iyy="0.1" iyz="0" izz="0.1"/>
+      <mass value="36.449"/>
+      <origin xyz="-0.100 0 -0.087" rpy="0 0 0"/>
+      <inertia ixx="2.792330" ixy="0" ixz="0" iyy="2.521060" iyz="0" izz="0.536551"/>
     </inertial>
   </xacro:macro>
   <property name="torso_damping" value="1"/>
-  <property name="torso_friction" value="0"/>
+  <property name="torso_friction" value="0.1"/>
   <property name="torso_effort" value="10000"/>
-  <property name="torso_velocity" value="10000"/>
-  <property name="torso_upper" value="0"/>
-  <property name="torso_lower" value="0.33"/>
+  <property name="torso_velocity" value="4.0"/>
+  <property name="torso_upper" value="0.33"/>
+  <property name="torso_lower" value="0"/>
 </robot>

File: ahl_robot/ahl_pr2_description/urdf/gripper/gripper.gazebo.xacro (robot description, xacro)
@@ -6,14 +6,4 @@
   <xacro:macro name="pr2_gripper_gazebo">
     <!-- left gripper -->
-    <gazebo reference="gripper_palm_l_link">
-      <gravity>1</gravity>
-      <maxVel>-1</maxVel>
-      <minDepth>0</minDepth>
-      <mu1>0</mu1>
-      <mu2>0</mu2>
-      <kp>10000000000.0</kp>
-      <kd>100000000.0</kd>
-      <selfCollide>1</selfCollide>
-    </gazebo>
     <gazebo reference="finger_ll_link">
       <gravity>1</gravity>
@@ -57,14 +47,4 @@
     </gazebo>
     <!-- left gripper -->
-    <gazebo reference="gripper_palm_r_link">
-      <gravity>1</gravity>
-      <maxVel>-1</maxVel>
-      <minDepth>0</minDepth>
-      <mu1>0</mu1>
-      <mu2>0</mu2>
-      <kp>10000000000.0</kp>
-      <kd>100000000.0</kd>
-      <selfCollide>1</selfCollide>
-    </gazebo>
     <gazebo reference="finger_rl_link">
       <gravity>1</gravity>

File: ahl_robot/ahl_pr2_description/urdf/gripper/gripper.property.xacro (robot description, xacro)
@@ -2,20 +2,4 @@
 <robot xmlns:xacro="http://ros.org/wiki/xacro">
   <property name="PI" value="3.1415926535897931"/>
-  <property name="gripper_palm_x" value="0"/>
-  <property name="gripper_palm_y" value="0"/>
-  <property name="gripper_palm_z" value="0"/>
-  <xacro:macro name="gripper_palm_inertial">
-    <inertial>
-      <mass value="1"/>
-      <origin xyz="0 0 0" rpy="0 0 0"/>
-      <inertia ixx="0.01" ixy="0" ixz="0" iyy="0.01" iyz="0" izz="0.01"/>
-    </inertial>
-  </xacro:macro>
-  <property name="gripper_palm_damping" value="1"/>
-  <property name="gripper_palm_friction" value="0"/>
-  <property name="gripper_palm_effort" value="10000"/>
-  <property name="gripper_palm_velocity" value="10000"/>
-  <property name="gripper_palm_upper" value="${M_PI / 2}"/>
-  <property name="gripper_palm_lower" value="${-M_PI / 2}"/>
   <property name="finger_x" value="0.0475"/>
   <property name="finger_y" value="0.01"/>
@@ -23,15 +7,15 @@
   <xacro:macro name="finger_inertial">
     <inertial>
-      <mass value="1"/>
-      <origin xyz="0 0 0" rpy="0 0 0"/>
-      <inertia ixx="0.01" ixy="0" ixz="0" iyy="0.01" iyz="0" izz="0.01"/>
+      <mass value="0.171"/>
+      <origin xyz="0.036 0 0" rpy="0 0 0"/>
+      <inertia ixx="0.0001" ixy="0" ixz="0" iyy="0.000197" iyz="0" izz="0.000181"/>
     </inertial>
   </xacro:macro>
   <property name="finger_damping" value="1"/>
-  <property name="finger_friction" value="0"/>
+  <property name="finger_friction" value="1"/>
   <property name="finger_effort" value="10000"/>
   <property name="finger_velocity" value="10000"/>
-  <property name="finger_upper" value="${M_PI / 2}"/>
-  <property name="finger_lower" value="${-M_PI / 2}"/>
+  <property name="finger_upper" value="0.548"/>
+  <property name="finger_lower" value="0"/>
   <property name="finger_tip_x" value="0.091"/>
   <property name="finger_tip_y" value="0.005"/>
@@ -39,14 +23,14 @@
   <xacro:macro name="finger_tip_inertial">
     <inertial>
-      <mass value="1"/>
-      <origin xyz="0 0 0" rpy="0 0 0"/>
-      <inertia ixx="0.01" ixy="0" ixz="0" iyy="0.01" iyz="0" izz="0.01"/>
+      <mass value="0.4419"/>
+      <origin xyz="0.004 0 0" rpy="0 0 0"/>
+      <inertia ixx="0.0001" ixy="0" ixz="0" iyy="0.0001" iyz="0" izz="0.0001"/>
     </inertial>
   </xacro:macro>
   <property name="finger_tip_damping" value="1"/>
-  <property name="finger_tip_friction" value="0"/>
+  <property name="finger_tip_friction" value="1"/>
   <property name="finger_tip_effort" value="10000"/>
   <property name="finger_tip_velocity" value="10000"/>
-  <property name="finger_tip_upper" value="${M_PI / 2}"/>
-  <property name="finger_tip_lower" value="${-M_PI / 2}"/>
+  <property name="finger_tip_upper" value="0.548"/>
+  <property name="finger_tip_lower" value="0"/>
 </robot>

File: ahl_robot/ahl_pr2_description/urdf/gripper/gripper.transmission.xacro (robot description, xacro)
@@ -6,14 +6,4 @@
   <xacro:macro name="pr2_gripper_transmission">
     <!-- left gripper -->
-    <transmission name="gripper_palm_l_trans">
-      <type>transmission_interface/SimpleTransmission</type>
-      <actuator name="gripper_palm_l_motor">
-        <hardwareInterface>EffortJointInterface</hardwareInterface>
-        <mechanicalReduction>1</mechanicalReduction>
-      </actuator>
-      <joint name="gripper_palm_l_joint">
-        <hardwareInterface>EffortJointInterface</hardwareInterface>
-      </joint>
-    </transmission>
     <transmission name="finger_ll_trans">
       <type>transmission_interface/SimpleTransmission</type>
@@ -57,14 +47,4 @@
     </transmission>
     <!-- right gripper -->
-    <transmission name="gripper_palm_r_trans">
-      <type>transmission_interface/SimpleTransmission</type>
-      <actuator name="gripper_palm_r_motor">
-        <hardwareInterface>EffortJointInterface</hardwareInterface>
-        <mechanicalReduction>1</mechanicalReduction>
-      </actuator>
-      <joint name="gripper_palm_r_joint">
-        <hardwareInterface>EffortJointInterface</hardwareInterface>
-      </joint>
-    </transmission>
     <transmission name="finger_rl_trans">
       <type>transmission_interface/SimpleTransmission</type>

Commit message: Modified wrong upper and lower values of arm.
Modified pr2.yaml. Now joint limit should be set properly.

File: ahl_robot/ahl_pr2_description/urdf/arm/arm.property.xacro (robot description, xacro)
@@ -96,6 +96,6 @@
   <property name="wrist_flex_effort" value="10000"/>
   <property name="wrist_flex_velocity" value="10000"/>
-  <property name="wrist_flex_upper" value="-2.180004"/>
-  <property name="wrist_flex_lower" value="0"/>
+  <property name="wrist_flex_upper" value="0"/>
+  <property name="wrist_flex_lower" value="-2.180004"/>
   <property name="wrist_roll_x" value="0.03"/>
   <property name="wrist_roll_y" value="0"/>

File: ahl_robot/ahl_pr2_description/urdf/gripper/gripper.property.xacro (robot description, xacro)
@@ -23,5 +23,5 @@
   <xacro:macro name="finger_tip_inertial">
     <inertial>
-      <mass value="0.04419"/>
+      <mass value="0.044"/>
       <origin xyz="0.004 0 0" rpy="0 0 0"/>
       <inertia ixx="0.00001" ixy="0" ixz="0" iyy="0.00001" iyz="0" izz="0.00001"/>

Commit message: Modified gravity compensation task.
Modified some control gains.

File: ahl_robot/ahl_pr2_description/urdf/arm/arm.property.xacro (robot description, xacro)
@@ -49,5 +49,6 @@
   <property name="upper_arm_velocity" value="10000"/>
   <property name="upper_arm_upper" value="3.900008"/>
-  <property name="upper_arm_lower" value="-0.800000"/>
+<!--  <property name="upper_arm_lower" value="-0.800000"/> -->
+  <property name="upper_arm_lower" value="-3.900008"/>
   <property name="elbow_x" value="0.28"/>
   <property name="elbow_y" value="0"/>
@@ -64,5 +65,5 @@
   <property name="elbow_effort" value="10000"/>
   <property name="elbow_velocity" value="10000"/>
-  <property name="elbow_upper" value="0"/>
+  <property name="elbow_upper" value="1.0"/>
   <property name="elbow_lower" value="-2.321305"/>
   <property name="forearm_x" value="0.09"/>
@@ -96,5 +97,5 @@
   <property name="wrist_flex_effort" value="10000"/>
   <property name="wrist_flex_velocity" value="10000"/>
-  <property name="wrist_flex_upper" value="0"/>
+  <property name="wrist_flex_upper" value="1.0"/>
   <property name="wrist_flex_lower" value="-2.180004"/>
   <property name="wrist_roll_x" value="0.03"/>

File: ahl_robot/ahl_pr2_description/urdf/base/base.property.xacro (robot description, xacro)
@@ -125,5 +125,5 @@
     </inertial>
   </xacro:macro>
-  <property name="torso_damping" value="10.0"/>
+  <property name="torso_damping" value="30.0"/>
   <property name="torso_friction" value="0.1"/>
   <property name="torso_effort" value="10000"/>

File: ahl_robot/ahl_pr2_description/urdf/gripper/gripper.property.xacro (robot description, xacro)
@@ -7,5 +7,5 @@
   <xacro:macro name="finger_inertial">
     <inertial>
-      <mass value="0.171"/>
+      <mass value="0.4"/>
       <origin xyz="0.036 0 0" rpy="0 0 0"/>
       <inertia ixx="0.0001" ixy="0" ixz="0" iyy="0.000197" iyz="0" izz="0.000181"/>
@@ -23,7 +23,7 @@
   <xacro:macro name="finger_tip_inertial">
     <inertial>
-      <mass value="0.044"/>
+      <mass value="0.4"/>
       <origin xyz="0.004 0 0" rpy="0 0 0"/>
-      <inertia ixx="0.00001" ixy="0" ixz="0" iyy="0.00001" iyz="0" izz="0.00001"/>
+      <inertia ixx="0.0001" ixy="0" ixz="0" iyy="0.0001" iyz="0" izz="0.0001"/>
     </inertial>
   </xacro:macro>
